File: boards/phono-power/phono-power.kicad_pcb (KiCad board)
At the start: 2 copper layers, 251.5 x 152.4 mm, 24 parts, among them J1 Conn_01x05, J2 Conn_01x06_Female, J3 Conn_01x06_Female, SW1 SW_SPST_GND, T1 Transformer_272X, U1 6CA4

Commit message: resize boards
Parts:
- T1: value Transformer_272X -> Hammond 272X
- moved F1 114.3 mm to (119.4, 66.0), turned to 270 degrees
- moved H4 82.9 mm to (194.3, 214.6)
- moved NE1 74.0 mm to (165.1, 209.6)
- moved H3 73.7 mm to (194.3, 31.8)
- moved J1 71.1 mm to (162.6, 43.2)
- moved R2 66.2 mm to (190.5, 204.5)
- moved C1 55.8 mm to (170.2, 57.1), turned to 180 degrees
- moved SW1 49.6 mm to (180.3, 201.9)
- moved H2 38.1 mm to (24.1, 214.6)
- moved R1 35.8 mm to (177.8, 57.1), turned to 0 degrees
- moved J2 34.3 mm to (39.4, 212.1)
- moved J3 34.3 mm to (95.2, 212.1)
- moved T1 30.9 mm to (162.6, 104.1)
- moved C2 29.9 mm to (133.3, 179.1)
- moved U1 19.4 mm to (163.8, 171.4)
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Other:
- board size 251.5 x 152.4 mm -> 177.8 x 190.5 mm
